File: pcb/esp_smart_clock/esp_smart_clock.kicad_sch (KiCad schematic)
At the start: 68 parts, among them IC1 CR1220-2, J1 Connector, USB-TYPE-C-16P, J10 MTLW-101-05-G-D-150, J11 MTLW-101-05-G-D-150, J14 MTLW-101-05-G-D-150, J15 MTLW-101-05-G-D-150, J16 MTLW-101-05-G-D-150, J17 MTLW-101-05-G-D-150, J18 MTLW-101-05-G-D-150, J19 MTLW-101-05-G-D-150, J2 MTLW-101-05-G-D-150, J20 MTLW-101-05-G-D-150, J22 MTLW-101-05-G-D-150, J23 MTLW-101-05-G-D-150, J24 MTLW-101-05-G-D-150, J3 MTLW-101-05-G-D-150, J4 MTLW-101-05-G-D-150, J5 MTLW-101-05-G-D-150, J6 MTLW-101-05-G-D-150, J7 MTLW-101-05-G-D-150, J8 MTLW-101-05-G-D-150, J9 MTLW-101-05-G-D-150, P1 PHR-2, P2 PHR-2, P3 PHR-2, Q1 S8050, Q2 S8050, Q3 S8050, Q4 S8050, U1 ESP32-WROOM-32D-N4, U2 AMS1117-3.3, U3 TP4056, U4 PCF8563T, U8 CH340K, X1 Q13FC1350000400

Commit message: Update README and PCB files, add SD card subproject
Updated the README with new ESP32 module info, BOM clarifications, and added a gallery section. Removed outdated PCB autosave and backup files, added new SD card KiCad project files, and updated main PCB and schematic files to reflect recent hardware changes.
Connections:
- net GND: now also U3.9 (EP); no longer U3.6 (STDBY#), U3.7 (CHRG#)
- no-connect marks 18 -> 22
Changed lines of the file:
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@@
 	)
 	(junction
-		(at 72.39 123.19)
-		(diameter 0)
-		(color 0 0 0 0)
-	)
-	(junction
 		(at 173.99 161.29)
 		(diameter 0)
@@
 	)
 	(no_connect
-		(at 88.9 130.81)
-	)
-	(no_connect
 		(at 68.58 66.04)
 	)
@@
 	)
 	(no_connect
+		(at 68.58 88.9)
+	)
+	(no_connect
 		(at 234.95 24.13)
 	)
@@
 	)
 	(no_connect
+		(at 109.22 58.42)
+	)
+	(no_connect
 		(at 68.58 83.82)
 	)
@@
 	)
 	(no_connect
+		(at 73.66 120.65)
+	)
+	(no_connect
+		(at 73.66 123.19)
+	)
+	(no_connect
 		(at 119.38 16.51)
 	)
@@
 		(at 153.67 191.77)
 	)
+	(no_connect
+		(at 68.58 50.8)
+	)
 	(wire
 		(pts
@@
 	(wire
 		(pts
-			(xy 73.66 120.65) (xy 72.39 120.65)
-		)
-		(stroke
-			(width 0)
-			(type default)
-		)
-	)
-	(wire
-		(pts
 			(xy 127 68.58) (xy 130.81 68.58)
 		)
@@
 	(wire
 		(pts
-			(xy 72.39 120.65) (xy 72.39 123.19)
-		)
-		(stroke
-			(width 0)
-			(type default)
-		)
-	)
-	(wire
-		(pts
 			(xy 130.81 161.29) (xy 152.4 161.29)
 		)
@@
 	(wire
 		(pts
-			(xy 72.39 123.19) (xy 72.39 125.73)
-		)
-		(stroke
-			(width 0)
-			(type default)
-		)
-	)
-	(wire
-		(pts
 			(xy 196.85 92.71) (xy 194.31 92.71)
 		)
@@
 	(wire
 		(pts
-			(xy 72.39 123.19) (xy 73.66 123.19)
-		)
-		(stroke
-			(width 0)
-			(type default)
-		)
-	)
-	(wire
-		(pts
 			(xy 123.19 161.29) (xy 123.19 163.83)
 		)
@@
 	)
 	(symbol
+		(lib_id "power:GND")
+		(at 88.9 130.81 0)
+		(unit 1)
+		(exclude_from_sim no)
+		(in_bom yes)
+		(on_board yes)
+		(dnp no)
+		(fields_autoplaced yes)
+		(property "Reference" "#PWR030"
+			(at 88.9 137.16 0)
+			(effects
+				(font
+					(size 1.27 1.27)
+				)
+				(hide yes)
+			)
+		)
+		(property "Value" "GND"
+			(at 88.9 135.89 0)
+			(effects
+				(font
+					(size 1.27 1.27)
+				)
+			)
+		)
+		(property "Footprint" ""
+			(at 88.9 130.81 0)
+			(effects
+				(font
+					(size 1.27 1.27)
+				)
+				(hide yes)
+			)
+		)
+		(property "Datasheet" ""
+			(at 88.9 130.81 0)
+			(effects
+				(font
+					(size 1.27 1.27)
+				)
+				(hide yes)
+			)
+		)
+		(property "Description" "Power symbol creates a global label with name \"GND\" , ground"
+			(at 88.9 130.81 0)
+			(effects
+				(font
+					(size 1.27 1.27)
+				)
+				(hide yes)
+			)
+		)
+		(pin "1"
+		)
+		(instances
+			(project "esp_smart_clock"
+				(path "/f9c2bea1-4efc-4a36-9f42-8207ef5de284"
+					(reference "#PWR030")
+					(unit 1)
+				)
+			)
+		)
+	)
+	(symbol
 		(lib_id "PCM_JLCPCB-Diodes:Switching,1N4148WS")
 		(at 238.76 114.3 270)
@@
 	)
 	(symbol
+		(lib_id "power:GND")
+		(at 166.37 143.51 90)
+		(unit 1)
+		(exclude_from_sim no)
+		(in_bom yes)
+		(on_board yes)
+		(dnp no)
+		(fields_autoplaced yes)
+		(property "Reference" "#PWR029"
+			(at 172.72 143.51 0)
+			(effects
+				(font
+					(size 1.27 1.27)
+				)
+				(hide yes)
+			)
+		)
+		(property "Value" "GND"
+			(at 170.18 143.5099 90)
+			(effects
+				(font
+					(size 1.27 1.27)
+				)
+				(justify right)
+			)
+		)
+		(property "Footprint" ""
+			(at 166.37 143.51 0)
+			(effects
+				(font
+					(size 1.27 1.27)
+				)
+				(hide yes)
+			)
+		)
+		(property "Datasheet" ""
+			(at 166.37 143.51 0)
+			(effects
+				(font
+					(size 1.27 1.27)
+				)
+				(hide yes)
+			)
+		)
+		(property "Description" "Power symbol creates a global label with name \"GND\" , ground"
+			(at 166.37 143.51 0)
+			(effects
+				(font
+					(size 1.27 1.27)
+				)
+				(hide yes)
+			)
+		)
+		(pin "1"
+		)
+		(instances
+			(project "esp_smart_clock"
+				(path "/f9c2bea1-4efc-4a36-9f42-8207ef5de284"
+					(reference "#PWR029")
+					(unit 1)
+				)
+			)
+		)
+	)
+	(symbol
 		(lib_id "MTLW-101-05-G-D-150:MTLW-101-05-G-D-150")
 		(at 163.83 68.58 0)
@@
 					(unit 1)
 				)
-			)
-		)
-	)
-	(symbol
-		(lib_id "power:GND")
-		(at 72.39 125.73 0)
-		(unit 1)
-		(exclude_from_sim no)
-		(in_bom yes)
-		(on_board yes)
-		(dnp no)
-		(fields_autoplaced yes)
-		(property "Reference" "#PWR023"
-			(at 72.39 132.08 0)
-			(effects
-				(font
-					(size 1.27 1.27)
-				)
-				(hide yes)
-			)
-		)
-		(property "Value" "GND"
-			(at 72.39 130.81 0)
-			(effects
-				(font
-					(size 1.27 1.27)
-				)
-			)
-		)
-		(property "Footprint" ""
-			(at 72.39 125.73 0)
-			(effects
-				(font
-					(size 1.27 1.27)
-				)
-				(hide yes)
-			)
-		)
-		(property "Datasheet" ""
-			(at 72.39 125.73 0)
-			(effects
-				(font
-					(size 1.27 1.27)
-				)
-				(hide yes)
-			)
-		)
-		(property "Description" "Power symbol creates a global label with name \"GND\" , ground"
-			(at 72.39 125.73 0)
-			(effects
-				(font
-					(size 1.27 1.27)
-				)
-				(hide yes)
-			)
-		)
-		(pin "1"
-		)
-		(instances
-			(project "esp_smart_clock"
-				(path "/f9c2bea1-4efc-4a36-9f42-8207ef5de284"
-					(reference "#PWR023")
-					(unit 1)
-				)

Commit message: Remove D2 diode and update net assignments
Removed the D2 (1N4148WS) diode footprint from the PCB design and updated net assignments throughout the esp_smart_clock.kicad_pcb file to reflect the change. Also updated backup files and made minor netlist adjustments, marking IO14 and IO16 as unconnected. Deleted old backup files and added new ones.
Parts:
- removed D10, D2: 1N4148WS, PCM_JLCPCB:D_SOD-323, symbol PCM_JLCPCB-Diodes:Switching,1N4148WS
- removed J14, J24: MTLW-101-05-G-D-150, footprints:SAMTEC_MTLW-101-05-G-D-150, symbol MTLW-101-05-G-D-150:MTLW-101-05-G-D-150
- removed Q1, Q4: S8050, PCM_JLCPCB:Q_SOT-23, symbol PCM_JLCPCB-Transistors:NPN,S8050
- removed R7, R8: 1.2kΩ, PCM_JLCPCB:R_0402, symbol PCM_JLCPCB-Resistors:0402,1.2kΩ
- added U5: W25Q128JVP, Package_SON:WSON-8-1EP_6x5mm_P1.27mm_EP3.4x4.3mm, symbol Memory_Flash:W25Q128JVP
Connections:
- net +3V3: now also U5.3 (~{WP}/IO_{2}), U5.7 (~{HOLD}/~{RESET}/IO_{3}), U5.8 (VCC)
- net GND: now also U5.4 (GND), U5.9 (EP)
- net IO14: now also U5.6 (CLK)
- net IO18: no longer J6.02
- net IO23: now also U5.5 (DI/IO_{0}); no longer J6.01
- net IO27: now also U5.1 (~{CS}); no longer J2.02
- net IO17: now reaches U1.28 (IO17)
- net IO17: now also J2.02
- net IO19: now reaches U1.31 (IO19)
- net IO19: now also U5.2 (DO/IO_{1})
- net IO21 renamed SDA
- net SDA: now also J6.01
- net IO22 renamed SCL
- net SCL: now also J6.02
- no-connect marks 22 -> 20
